Commit message: chassis size Change from Hoyuko into rplidar

File: Workspace/src/tinker_description_nav_only/urdf/tinker.urdf.xacro (robot description, xacro)
@@ -12,5 +12,5 @@
             <origin xyz="${stl_trans_xyz}" rpy="${stl_rotate_rpy}" />
             <geometry>
-                <mesh filename="package://tinker_description/meshes/tinker_base.stl" scale="${stl_viz_scale}" />
+                <mesh filename="package://tinker_description_nav_only/meshes/tinker_base.stl" scale="${stl_viz_scale}" />
             </geometry>
             <material name="">
@@ -21,15 +21,15 @@
             <origin xyz="${stl_trans_xyz}" rpy="${stl_rotate_rpy}" />
             <geometry>
-                <mesh filename="package://tinker_description/meshes/tinker_base.stl" scale="${stl_viz_scale}" />
+                <mesh filename="package://tinker_description_nav_only/meshes/tinker_base.stl" scale="${stl_viz_scale}" />
             </geometry>
         </collision>
     </link>
     <!-- laser -->
-    <xacro:property name="urg_front_trans_xyz" value="0.25 0. 0.25" />
-    <link name="urg_laser_front" />
-    <joint name="base_to_urg_front" type="fixed">
+    <xacro:property name="laser_trans_xyz" value="0.25 0. 0.25" />
+    <link name="laser" />
+    <joint name="base_to_laser" type="fixed">
         <parent link="base_link" />
-        <child link="urg_laser_front" />
-        <origin xyz="${urg_front_trans_xyz}" />
+        <child link="laser" />
+        <origin xyz="${laser_trans_xyz}" />
     </joint>
 </robot>

Commit message: rgbd pointcloud2 added

File: Workspace/src/tinker_description_nav_only/urdf/tinker.urdf.xacro (robot description, xacro)
@@ -33,3 +33,21 @@
         <origin xyz="${laser_trans_xyz}" />
     </joint>
+    <!-- rgbd camera -->
+    <link name="camera_depth_optical_frame">
+        <visual>
+            <geometry>
+                <box size="0.03 0.12 0.02" />
+            </geometry>
+            <origin xyz="0 0 0" rpy="0 0 0" />
+            <material name="blue">
+                <color rgba="0 0 0.8 0.5" />
+            </material>
+        </visual>
+    </link>
+        <joint name="base_to_camera" type="fixed">
+        <parent link="base_link" />
+        <child link="camera_depth_optical_frame" />
+        <origin xyz="-0.225 0 1.16" rpy="-2.0944 0 -1.5707" />
+        <axis xyz="0 0 1" />
+    </joint>
 </robot>

Commit message: rgbd pointcloud

File: Workspace/src/tinker_description_nav_only/urdf/tinker.urdf.xacro (robot description, xacro)
@@ -34,4 +34,5 @@
     </joint>
     <!-- rgbd camera -->
+    <xacro:property name="camera_depth_optical_frame_trans_xyz" value="-0.225 0 1.16" />
     <link name="camera_depth_optical_frame">
         <visual>

Commit message: update

File: Workspace/src/tinker_description_nav_only/urdf/tinker.urdf.xacro (robot description, xacro)
@@ -31,9 +31,9 @@
         <parent link="base_link" />
         <child link="laser" />
-        <origin xyz="${laser_trans_xyz}" />
+        <origin xyz="${laser_trans_xyz}" rpy="0 0 -0.7854"/>
     </joint>
     <!-- rgbd camera -->
-    <xacro:property name="camera_depth_optical_frame_trans_xyz" value="-0.225 0 1.16" />
-    <link name="camera_depth_optical_frame">
+    <xacro:property name="camera_link_trans_xyz" value="-0.225 0 1.32" />
+    <link name="camera_link">
         <visual>
             <geometry>
@@ -46,8 +46,8 @@
         </visual>
     </link>
-        <joint name="base_to_camera" type="fixed">
+        <joint name="base_to_camera_link" type="fixed">
         <parent link="base_link" />
-        <child link="camera_depth_optical_frame" />
-        <origin xyz="-0.225 0 1.16" rpy="-2.0944 0 -1.5707" />
+        <child link="camera_link" />
+        <origin xyz="-0.225 0 1.32" rpy="-3.14159 -3.14159 -3.14159" />
         <axis xyz="0 0 1" />
     </joint>

Commit message: camera .dae added (temporarily using d35.dea), rpy of the camera changed

File: Workspace/src/tinker_description_nav_only/urdf/tinker.urdf.xacro (robot description, xacro)
@@ -38,7 +38,8 @@
         <visual>
             <geometry>
-                <box size="0.03 0.12 0.02" />
+                <!--box size="0.03 0.12 0.02" /-->
+                <mesh filename="package://tinker_description_nav_only/meshes/d435.dae"/>
             </geometry>
-            <origin xyz="0 0 0" rpy="0 0 0" />
+            <origin xyz="0 0 0" rpy="0.9983 0 -1.5707" />
             <material name="blue">
                 <color rgba="0 0 0.8 0.5" />
@@ -48,6 +49,6 @@
         <joint name="base_to_camera_link" type="fixed">
         <parent link="base_link" />
-        <child link="camera_link" />
-        <origin xyz="-0.225 0 1.32" rpy="-3.14159 -3.14159 -3.14159" />
+        <child link="camera_link" />0.2618
+        <origin xyz="-0.225 0 1.32" rpy="-3.14159 -3.64075 -3.14159" />
         <axis xyz="0 0 1" />
     </joint>

Commit message: camera .dae added (temporarily using d35.dea), rpy of the camera changed

File: Workspace/src/tinker_description_nav_only/urdf/tinker.urdf.xacro (robot description, xacro)
@@ -49,5 +49,5 @@
         <joint name="base_to_camera_link" type="fixed">
         <parent link="base_link" />
-        <child link="camera_link" />0.2618
+        <child link="camera_link" />
         <origin xyz="-0.225 0 1.32" rpy="-3.14159 -3.64075 -3.14159" />
         <axis xyz="0 0 1" />

Commit message: rtabmap with imu & visual odom added

File: Workspace/src/tinker_description_nav_only/urdf/tinker.urdf.xacro (robot description, xacro)
@@ -1,4 +1,5 @@
 <?xml version="1.0" encoding="UTF-8"?>
 <robot xmlns:xacro="http://www.ros.org/wiki/xacro" name="tinker">
+    <xacro:property name="PI" value="3.1415926535897931" />
     <material name="black">
         <color rgba="0.1 0.1 0.1 1.0" />
@@ -25,4 +26,10 @@
         </collision>
     </link>
+    <link name="odom"/>
+    <joint name="base_to_odom" type="continuous">
+        <parent link="odom" />
+        <child link="base_link" />
+        <origin xyz="0 0 0" rpy="0 0 0"/>
+    </joint>
     <!-- laser -->
     <xacro:property name="laser_trans_xyz" value="0.25 0. 0.25" />
@@ -34,22 +41,111 @@
     </joint>
     <!-- rgbd camera -->
+    <!-- The following values are approximate, and the camera node
+     publishing TF values with actual calibrated camera extrinsic values -->
+    <xacro:property name="d435_cam_depth_to_infra1_offset" value="0.0"/>
+    <xacro:property name="d435_cam_depth_to_infra2_offset" value="-0.050"/>
+    <xacro:property name="d435_cam_depth_to_color_offset" value="0.015"/>
+    <!-- The following values model the aluminum peripherial case for the
+  	D435 camera, with the camera joint represented by the actual
+  	peripherial camera tripod mount -->
+    <xacro:property name="d435_cam_width" value="0.090"/>
+    <xacro:property name="d435_cam_height" value="0.025"/>
+    <xacro:property name="d435_cam_depth" value="0.02505"/>
+    <xacro:property name="d435_cam_mount_from_center_offset" value="0.0149"/>
+    <!-- glass cover is 0.1 mm inwards from front aluminium plate -->
+    <xacro:property name="d435_glass_to_front" value="0.1e-3"/>
+    <!-- see datasheet Revision 007, Fig. 4-4 page 65 -->
+    <xacro:property name="d435_zero_depth_to_glass" value="4.2e-3"/>
+    <!-- convenience precomputation to avoid clutter-->
+    <xacro:property name="d435_mesh_x_offset" value="${d435_cam_mount_from_center_offset-d435_glass_to_front-d435_zero_depth_to_glass}"/>
+    <!-- The following offset is relative the the physical D435 camera peripherial
+  	camera tripod mount -->
+    <xacro:property name="d435_cam_depth_px" value="${d435_cam_mount_from_center_offset}"/>
+    <xacro:property name="d435_cam_depth_py" value="0.0175"/>
+    <xacro:property name="d435_cam_depth_pz" value="${d435_cam_height/2}"/>
     <xacro:property name="camera_link_trans_xyz" value="-0.225 0 1.32" />
     <link name="camera_link">
-        <visual>
-            <geometry>
-                <!--box size="0.03 0.12 0.02" /-->
-                <mesh filename="package://tinker_description_nav_only/meshes/d435.dae"/>
-            </geometry>
-            <origin xyz="0 0 0" rpy="0.9983 0 -1.5707" />
-            <material name="blue">
-                <color rgba="0 0 0.8 0.5" />
-            </material>
-        </visual>
+      <origin xyz="0 0 0" rpy="${-PI/180*28.6} 0 ${-PI/4}" />
+      <xacro:include filename="$(find tinker_description_nav_only)/urdf/_d435.urdf.xacro"/>
     </link>
-        <joint name="base_to_camera_link" type="fixed">
+    <joint name="base_to_camera_link" type="fixed">
         <parent link="base_link" />
         <child link="camera_link" />
-        <origin xyz="-0.225 0 1.32" rpy="-3.14159 -3.64075 -3.14159" />
+        <origin xyz="${camera_link_trans_xyz}" rpy="${-PI} -3.64075 ${-PI}" />
         <axis xyz="0 0 1" />
     </joint>
+    <joint name="camera_depth_joint" type="fixed">
+        <origin xyz="0 0 0" rpy="0 0 0"/>
+        <parent link="camera_link"/>
+        <child link="camera_depth_frame" />
+      </joint>
+      <link name="camera_depth_frame"/>
+      <joint name="camera_depth_optical_joint" type="fixed">
+        <origin xyz="0 0 0" rpy="${-PI/2} 0 ${-PI/2}" />
+        <parent link="camera_depth_frame" />
+        <child link="camera_depth_optical_frame" />
+      </joint>
+      <link name="camera_depth_optical_frame"/>
+      <!-- camera left IR joints and links -->
+      <joint name="camera_infra1_joint" type="fixed">
+        <origin xyz="0 ${d435_cam_depth_to_infra1_offset} 0" rpy="0 0 0" />
+        <parent link="camera_link" />
+        <child link="camera_infra1_frame" />
+      </joint>
+      <link name="camera_infra1_frame"/>
+      <joint name="camera_infra1_optical_joint" type="fixed">
+        <origin xyz="0 0 0" rpy="${-PI/2} 0 ${-PI/2}" />
+        <parent link="camera_infra1_frame" />
+        <child link="camera_infra1_optical_frame" />
+      </joint>
+      <link name="camera_infra1_optical_frame"/>
+      <!-- camera right IR joints and links -->
+      <joint name="camera_infra2_joint" type="fixed">
+        <origin xyz="0 ${d435_cam_depth_to_infra2_offset} 0" rpy="0 0 0" />
+        <parent link="camera_link" />
+        <child link="camera_infra2_frame" />
+      </joint>
+      <link name="camera_infra2_frame"/>
+      <joint name="camera_infra2_optical_joint" type="fixed">
+        <origin xyz="0 0 0" rpy="${-PI/2} 0 ${-PI/2}" />
+        <parent link="camera_infra2_frame" />
+        <child link="camera_infra2_optical_frame" />
+      </joint>
+      <link name="camera_infra2_optical_frame"/>
+      <!-- camera color joints and links -->
+      <joint name="camera_color_joint" type="fixed">
+        <origin xyz="0 ${d435_cam_depth_to_color_offset} 0" rpy="0 0 0" />
+        <parent link="camera_link" />
+        <child link="camera_color_frame" />
+      </joint>
+      <link name="camera_color_frame"/>
+      <joint name="camera_color_optical_joint" type="fixed">
+        <origin xyz="0 0 0" rpy="${-PI/2} 0 ${-PI/2}" />
+        <parent link="camera_color_frame" />
+        <child link="camera_color_optical_frame" />
+      </joint>
+      <link name="camera_color_optical_frame"/>
+      <!-- camera imu -->
+    <link name="imu_optical_frame">
+	<origin xyz="0 0 0" rpy="0.9983 0 -1.5707" />
+	<xacro:include filename="$(find realsense2_description)/urdf/_d435i_imu_modules.urdf.xacro"/>
+    </link>
+    <joint name="base_to_imu_link" type="fixed">
+        <parent link="base_link" />
+        <child link="imu_optical_frame" />
+        <origin xyz="${camera_link_trans_xyz}" rpy="-3.14159 -3.64075 -3.14159" />
+        <axis xyz="0 0 0" />
+    </joint>
+      <link name="camera_accel_frame" />
+      <link name="camera_accel_optical_frame" />
+      <joint name="camera_accel_joint" type="fixed">
+        <origin xyz = "-0.01174 -0.00552 0.0051" rpy = "0 0 0" />
+        <parent link="imu_optical_frame" />
+        <child link="camera_accel_frame" />
+      </joint>
+      <joint name="camera_accel_optical_joint" type="fixed">
+        <origin xyz = "0 0 0" rpy = "${-PI/2} 0 ${-PI/2}" />
+        <parent link="camera_accel_frame" />
+        <child link="camera_accel_optical_frame" />
+      </joint>
 </robot>
