Commit message: change name tinker_description

File: Workspace/src/tinker_description/urdf/tinker.urdf.xacro (robot description, xacro)
@@ -13,5 +13,5 @@
             <origin xyz="${stl_trans_xyz}" rpy="${stl_rotate_rpy}" />
             <geometry>
-                <mesh filename="package://tinker_description_nav_only/meshes/tinker_base.stl" scale="${stl_viz_scale}" />
+                <mesh filename="package://tinker_description/meshes/tinker_base.stl" scale="${stl_viz_scale}" />
             </geometry>
             <material name="">
@@ -22,5 +22,5 @@
             <origin xyz="${stl_trans_xyz}" rpy="${stl_rotate_rpy}" />
             <geometry>
-                <mesh filename="package://tinker_description_nav_only/meshes/tinker_base.stl" scale="${stl_viz_scale}" />
+                <mesh filename="package://tinker_description/meshes/tinker_base.stl" scale="${stl_viz_scale}" />
             </geometry>
         </collision>
@@ -67,5 +67,5 @@
     <link name="camera_link">
       <origin xyz="0 0 0" rpy="${-PI/180*28.6} 0 ${-PI/4}" />
-      <xacro:include filename="$(find tinker_description_nav_only)/urdf/_d435.urdf.xacro"/>
+      <xacro:include filename="$(find tinker_description)/urdf/_d435.urdf.xacro"/>
     </link>
     <joint name="base_to_camera_link" type="fixed">
@@ -131,8 +131,8 @@
 	<xacro:include filename="$(find realsense2_description)/urdf/_d435i_imu_modules.urdf.xacro"/>
     </link>
-    <joint name="base_to_imu_link" type="fixed">
-        <parent link="base_link" />
+    <joint name="camera_to_imu_link" type="fixed">
+        <parent link="camera_link" />
         <child link="imu_optical_frame" />
-        <origin xyz="${camera_link_trans_xyz}" rpy="-3.14159 -3.64075 -3.14159" />
+        <origin xyz="0 0 0" rpy="0 0 0" />
         <axis xyz="0 0 0" />
     </joint>

Commit message: rtabmap obstacle_detection in voxels

File: Workspace/src/tinker_description/urdf/tinker.urdf.xacro (robot description, xacro)
@@ -126,26 +126,3 @@
       </joint>
       <link name="camera_color_optical_frame"/>
-      <!-- camera imu -->
-    <link name="imu_optical_frame">
-	<origin xyz="0 0 0" rpy="0.9983 0 -1.5707" />
-	<xacro:include filename="$(find realsense2_description)/urdf/_d435i_imu_modules.urdf.xacro"/>
-    </link>
-    <joint name="camera_to_imu_link" type="fixed">
-        <parent link="camera_link" />
-        <child link="imu_optical_frame" />
-        <origin xyz="0 0 0" rpy="0 0 0" />
-        <axis xyz="0 0 0" />
-    </joint>
-      <link name="camera_accel_frame" />
-      <link name="camera_accel_optical_frame" />
-      <joint name="camera_accel_joint" type="fixed">
-        <origin xyz = "-0.01174 -0.00552 0.0051" rpy = "0 0 0" />
-        <parent link="imu_optical_frame" />
-        <child link="camera_accel_frame" />
-      </joint>
-      <joint name="camera_accel_optical_joint" type="fixed">
-        <origin xyz = "0 0 0" rpy = "${-PI/2} 0 ${-PI/2}" />
-        <parent link="camera_accel_frame" />
-        <child link="camera_accel_optical_frame" />
-      </joint>
 </robot>

Commit message: unnecessary launch deleted

File: Workspace/src/tinker_description/urdf/tinker.urdf.xacro (robot description, xacro)
@@ -38,5 +38,5 @@
         <parent link="base_link" />
         <child link="laser" />
-        <origin xyz="${laser_trans_xyz}" rpy="0 0 -0.7854"/>
+        <origin xyz="${laser_trans_xyz}" rpy="0 0 ${-PI/4}"/>
     </joint>
     <!-- rgbd camera -->
@@ -67,10 +67,10 @@
     <link name="camera_link">
       <origin xyz="0 0 0" rpy="${-PI/180*28.6} 0 ${-PI/4}" />
-      <xacro:include filename="$(find tinker_description)/urdf/_d435.urdf.xacro"/>
+      <xacro:include filename="$(find realsense2_description)/urdf/_d435.urdf.xacro"/>
     </link>
     <joint name="base_to_camera_link" type="fixed">
         <parent link="base_link" />
         <child link="camera_link" />
-        <origin xyz="${camera_link_trans_xyz}" rpy="${-PI} -3.64075 ${-PI}" />
+        <origin xyz="${camera_link_trans_xyz}" rpy="${-PI} ${-PI/180*208.6} ${-PI}" />
         <axis xyz="0 0 1" />
     </joint>

Commit message: delete files

File: Workspace/src/tinker_description/urdf/tinker.urdf.xacro (robot description, xacro)
@@ -38,5 +38,5 @@
         <parent link="base_link" />
         <child link="laser" />
-        <origin xyz="${laser_trans_xyz}" rpy="0 0 ${-PI/4}"/>
+        <origin xyz="${laser_trans_xyz}" rpy="0 0 ${-PI}"/>
     </joint>
     <!-- rgbd camera -->
